Commit message: new mujoco models

File: mujoco-setup/assembly_bala2ish/urdf/assembly_bala2ish.urdf (robot description, URDF)
Before this commit: robot assembly_bala2ish, 5 links, 4 joints
Links:
- added link mark_wheel, mass 3.39412e-08; visual mesh filename=package://assembly_bala2ish/meshes/mark_wheel.stl scale=1 1 1
- added link mark_wheel_1, mass 3.39412e-08; visual mesh filename=package://assembly_bala2ish/meshes/mark_wheel.stl scale=1 1 1
Joints:
- added joint fastened_3: type fixed, parent wheel_1, child mark_wheel_1, origin xyz=-0.01415 2.17403e-34 3.46945e-18 rpy=-3.03858e-64 1.75162e-46 -8.75812e-47, axis -1 -3.20732e-48 -2.1684e-16
- added joint fastened_4: type fixed, parent wheel, child mark_wheel, origin xyz=0.01415 -2.17403e-34 3.46945e-18 rpy=2.73691e-48 2.1684e-16 -3.14159, axis -1 -3.20732e-48 -2.1684e-16
- joint fastened_2: origin xyz=0.008 0.0175 0.0625 rpy=0 -0 0 -> xyz=0.008 0.0225 0.0625 rpy=0 -0 0
- joint wheel_right: axis 1 -0 -0 -> -1 -3.20732e-48 -2.1684e-16; origin xyz=0.031 -1.73472e-18 0.0225 rpy=-3.14159 1.91478e-96 -3.14159 -> xyz=0.031 5.98699e-49 0.0225 rpy=-6.74701e-80 2.1684e-16 -3.20732e-48

File: mujoco-setup/assembly_simplified/urdf/assembly_simplified.urdf (robot description, URDF)
Before this commit: robot assembly_simplified, 8 links, 7 joints
Links:
- removed link sketch_9__1_
- added link mark_wheel, mass 3.39412e-08; visual mesh filename=package://assembly_simplified/meshes/mark_wheel.stl scale=1 1 1
- added link mark_wheel_1, mass 3.39412e-08; visual mesh filename=package://assembly_simplified/meshes/mark_wheel.stl scale=1 1 1
Joints:
- added joint fastened_6: type fixed, parent wheel, child mark_wheel, origin xyz=0.01415 -4.34805e-34 3.46945e-18 rpy=6.95476e-64 2.1684e-16 -3.14159, axis -1 -3.20732e-48 -2.1684e-16
- joint fastened_5: axis 0 0 1 -> -1 -3.20732e-48 -2.1684e-16; child sketch_9__1_ -> mark_wheel_1; origin xyz=0 0 0 rpy=0 -0 0 -> xyz=-0.01415 -3.45509e-33 -3.46945e-18 rpy=-3.14159 -4.33681e-16 -1.03455e-45; parent root -> wheel_1
- joint wheel_left: axis 1 3.20732e-48 2.1684e-16 -> -1 -0 -0; origin xyz=-0.02765 0 0.0225 rpy=3.14159 -2.0349e-16 -5.54453e-18 -> xyz=-0.02765 -1.1074e-31 0.0225 rpy=3.14159 9.80909e-45 -4.2039e-45; parent sketch_9__1_ -> motor_base
- joint wheel_right: axis 1 3.20732e-48 2.1684e-16 -> -1 -3.20732e-48 -2.1684e-16; origin xyz=0.02765 0 0.0225 rpy=3.14159 -2.31296e-16 -3.14159 -> xyz=0.02765 2.17403e-34 0.0225 rpy=0 2.1684e-16 -3.20732e-48; parent sketch_9__1_ -> motor_base
