Commit message: bala2ish

File: mujoco-setup/assembly_simplified_long/urdf/assembly_simplified_long.urdf (robot description, URDF)
Before this commit: robot assembly_simplified, 8 links, 7 joints
Links:
- link electronics: mass 0.0319999 -> 0.0658623; geometry visual mesh filename=package://assembly_simplified_long/meshes/Electronics.stl scale=1 1 1
- link lipos: mass 0.040025 -> 0.0930383; geometry visual mesh filename=package://assembly_simplified_long/meshes/Lipos.stl scale=1 1 1
- link motor_base: geometry visual mesh filename=package://assembly_simplified_long/meshes/Motor_base.stl scale=1 1 1
- link sensor_imu: geometry visual mesh filename=package://assembly_simplified_long/meshes/sensor_imu.stl scale=1 1 1
- link wheel: geometry visual mesh filename=package://assembly_simplified_long/meshes/Wheel.stl scale=1 1 1
- link wheel_1: geometry visual mesh filename=package://assembly_simplified_long/meshes/Wheel.stl scale=1 1 1
Joints:
- joint fastened_2: origin xyz=-4.50423e-18 -1.35525e-18 0.0395128 rpy=1.35525e-16 6.93335e-33 0 -> xyz=0 -3.87602e-18 0.0395128 rpy=1.35525e-16 6.93335e-33 0
- joint fastened_3: origin xyz=2.67866e-18 -3.20291e-18 0.01525 rpy=-2.46519e-32 -6.93335e-33 9.39644e-49 -> xyz=-1.73472e-18 -6.82138e-19 0.01525 rpy=-2.46519e-32 -6.93335e-33 9.39644e-49
- joint fastened_4: origin xyz=0.013 0.007 0.0162 rpy=0 -0 0 -> xyz=0.013 -0.013 0.0162 rpy=0 -0 0

File: mujoco-setup/assembly_simplified_tall/urdf/assembly_simplified_tall.urdf (robot description, URDF)
Before this commit: robot assembly_simplified, 8 links, 7 joints
Links:
- link electronics: mass 0.0319999 -> 0.071506; geometry visual mesh filename=package://assembly_simplified_tall/meshes/Electronics.stl scale=1 1 1
- link lipos: geometry visual mesh filename=package://assembly_simplified_tall/meshes/Lipos.stl scale=1 1 1
- link motor_base: geometry visual mesh filename=package://assembly_simplified_tall/meshes/Motor_base.stl scale=1 1 1
- link sensor_imu: geometry visual mesh filename=package://assembly_simplified_tall/meshes/sensor_imu.stl scale=1 1 1
- link wheel: geometry visual mesh filename=package://assembly_simplified_tall/meshes/Wheel.stl scale=1 1 1
- link wheel_1: geometry visual mesh filename=package://assembly_simplified_tall/meshes/Wheel.stl scale=1 1 1
Joints:
- joint fastened_4: origin xyz=0.013 0.007 0.0162 rpy=0 -0 0 -> xyz=0.013 0.007 0.0362 rpy=0 -0 0
