Commit message: mujoco model updates

File: mujoco-setup/assembly_simplified/urdf/assembly_simplified.urdf (robot description, URDF)
Before this commit: robot assembly_simplified, 9 links, 8 joints
Links:
- added link sketch_wheelbase__1_, mass 1e-09
- link mark_wheel: mass 3.39412e-08 -> 4.38412e-08
- link mark_wheel_1: mass 3.39412e-08 -> 4.38412e-08
- link wheel: mass 0.0281308 -> 0.0435645
- link wheel_1: mass 0.0281308 -> 0.0435645
Joints:
- added joint fastened_2_1: type fixed, parent motor_base, child lipos, origin xyz=0 -3.87602e-18 0.0450128 rpy=1.35525e-16 6.93335e-33 0, axis -1.13185e-16 -2.46519e-32 -1
- joint fastened_2: axis -1.13185e-16 -2.46519e-32 -1 -> 0 0 1; child lipos -> sketch_wheelbase__1_; origin xyz=-4.50423e-18 -1.35525e-18 0.0395128 rpy=1.35525e-16 6.93335e-33 0 -> xyz=0 0 0 rpy=0 -0 0; parent motor_base -> root
- joint fastened_3: origin xyz=2.67866e-18 -3.20291e-18 0.01525 rpy=-2.46519e-32 -6.93335e-33 9.39644e-49 -> xyz=-1.73472e-18 -8.98979e-19 0.01525 rpy=-2.46519e-32 -6.93335e-33 9.39644e-49
- joint fastened_5: origin xyz=-0.01415 -3.45509e-33 -3.46945e-18 rpy=-3.14159 -4.33681e-16 -1.03455e-45 -> xyz=-0.01415 2.70546e-34 0 rpy=-3.14159 -4.33681e-16 3.50325e-45
- joint fastened_6: origin xyz=0.01415 -4.34805e-34 3.46945e-18 rpy=6.95476e-64 2.1684e-16 -3.14159 -> xyz=0.01415 -2.70546e-34 1.04083e-17 rpy=6.95476e-64 2.1684e-16 -3.14159
- joint wheel_left: axis -1 -0 -0 -> 1 0 0; origin xyz=-0.02765 -1.1074e-31 0.0225 rpy=3.14159 9.80909e-45 -4.2039e-45 -> xyz=-0.02765 0 0.028 rpy=3.14159 4.2039e-44 -1.82169e-44; parent motor_base -> sketch_wheelbase__1_
- joint wheel_right: origin xyz=0.02765 2.17403e-34 0.0225 rpy=0 2.1684e-16 -3.20732e-48 -> xyz=0.02765 0 0.028 rpy=0 2.1684e-16 -3.20732e-48; parent motor_base -> sketch_wheelbase__1_
